File: deepad_schem_and_pcb/myHackpad.kicad_pcb (KiCad board)
At the start: 2 copper layers, 73.8 x 59.5 mm, 17 parts, among them J1 OLED Display Pin, SW1 SW_Push_45deg, SW2 SW_Push_45deg, SW3 SW_Push_45deg, SW4 SW_Push_45deg, SW5 SW_Push_45deg, SW7 RotaryEncoder_Switch, U1 MOUDLE-SEEEDUINO-XIAO

Commit message: added all files
Parts:
- moved SW7 1.50 mm to (106.8, 72.3)
Routing:
- net ROW 1: track 74.7 -> 178.8 mm
- net COL 1: track 154.1 -> 74.5 mm, vias 0 -> 1
- net EC11A: track 82.0 -> 79.9 mm
- net GND: track 125.6 -> 127.4 mm, vias 9 -> 8
- net EC11SWB: track 5.74 -> 4.49 mm
- net EC11B: track 56.5 -> 57.5 mm
Other:
- board size 73.8 x 59.5 mm -> 75.2 x 59.6 mm
